File: LSE.kicad_sch (KiCad schematic)
At the start: 5 parts, among them Y501 32.758kHz

Commit message: ongoing.
Parts:
- R501: value 0 -> 0k
Changed lines of the file:
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@@
 			)
 		)
-		(property "Value" "0"
+		(property "Value" "0k"
 			(at 135.128 86.614 0)
 			(effects
@@
 			)
 		)
-		(property "Datasheet" "~"
+		(property "Datasheet" "https://www.microcrystal.com/fileadmin/Media/Products/32kHz/Datasheet/CM9V-T1A.pdf"
 			(at 120.65 95.25 0)
 			(effects
