File: power.kicad_sch (KiCad schematic)
At the start: 10 parts

Commit message: ongoing.
Parts:
- gave numbers to parts that had none: 9
- renumbered BT1 to BT101
Changed lines of the file:
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@@
 		(dnp no)
 		(fields_autoplaced yes)
-		(property "Reference" "#PWR?"
+		(property "Reference" "#PWR0108"
 			(at 121.92 120.65 0)
 			(effects
@@
 			(project "multiplexI2C"
 				(path "/0c2d0c14-8850-4a30-bb78-b2f40cb442ba/872e59d9-aae9-4a0c-a438-0cad18134c8d"
-					(reference "#PWR?")
+					(reference "#PWR0108")
 					(unit 1)
 				)
@@
 		(on_board yes)
 		(dnp no)
-		(property "Reference" "U?"
+		(property "Reference" "U101"
 			(at 159.512 81.534 0)
 			(effects
@@
 			(project "multiplexI2C"
 				(path "/0c2d0c14-8850-4a30-bb78-b2f40cb442ba/872e59d9-aae9-4a0c-a438-0cad18134c8d"
-					(reference "U?")
+					(reference "U101")
 					(unit 1)
 				)
@@
 		(on_board yes)
 		(dnp no)
-		(property "Reference" "#FLG?"
+		(property "Reference" "#FLG0101"
 			(at 145.415 59.69 0)
 			(effects
@@
 			(project "multiplexI2C"
 				(path "/0c2d0c14-8850-4a30-bb78-b2f40cb442ba/872e59d9-aae9-4a0c-a438-0cad18134c8d"
-					(reference "#FLG?")
+					(reference "#FLG0101")
 					(unit 1)
 				)
@@
 		(dnp no)
 		(fields_autoplaced yes)
-		(property "Reference" "#PWR?"
+		(property "Reference" "#PWR0105"
 			(at 152.4 50.8 0)
 			(effects
@@
 			(project "multiplexI2C"
 				(path "/0c2d0c14-8850-4a30-bb78-b2f40cb442ba/872e59d9-aae9-4a0c-a438-0cad18134c8d"
-					(reference "#PWR?")
+					(reference "#PWR0105")
 					(unit 1)
 				)
@@
 		(on_board yes)
 		(dnp no)
-		(property "Reference" "C?"
+		(property "Reference" "C105"
 			(at 111.76 97.79 0)
 			(effects
@@
 			(project "multiplexI2C"
 				(path "/0c2d0c14-8850-4a30-bb78-b2f40cb442ba/872e59d9-aae9-4a0c-a438-0cad18134c8d"
-					(reference "C?")
+					(reference "C105")
 					(unit 1)
 				)
@@
 		(on_board yes)
 		(dnp no)
-		(property "Reference" "C?"
+		(property "Reference" "C104"
 			(at 102.87 97.79 0)
 			(effects
@@
 			(project "multiplexI2C"
 				(path "/0c2d0c14-8850-4a30-bb78-b2f40cb442ba/872e59d9-aae9-4a0c-a438-0cad18134c8d"
-					(reference "C?")
+					(reference "C104")
 					(unit 1)
 				)
@@
 		(on_board yes)
 		(dnp no)
-		(property "Reference" "BT?"
+		(property "Reference" "BT101"
 			(at 163.83 120.0784 0)
 			(effects
@@
 				)
 				(path "/0c2d0c14-8850-4a30-bb78-b2f40cb442ba/872e59d9-aae9-4a0c-a438-0cad18134c8d"
-					(reference "BT?")
+					(reference "BT101")
 					(unit 1)
 				)
@@
 		(on_board yes)
 		(dnp no)
-		(property "Reference" "J?"
+		(property "Reference" "J101"
 			(at 155.702 67.056 90)
 			(effects
@@
 			(project "multiplexI2C"
 				(path "/0c2d0c14-8850-4a30-bb78-b2f40cb442ba/872e59d9-aae9-4a0c-a438-0cad18134c8d"
-					(reference "J?")
+					(reference "J101")
 					(unit 1)
 				)
@@
 		(dnp no)
 		(fields_autoplaced yes)
-		(property "Reference" "#PWR?"
+		(property "Reference" "#PWR0107"
 			(at 156.21 109.22 0)
 			(effects
@@
 			(project "multiplexI2C"
 				(path "/0c2d0c14-8850-4a30-bb78-b2f40cb442ba/872e59d9-aae9-4a0c-a438-0cad18134c8d"
-					(reference "#PWR?")
+					(reference "#PWR0107")
 					(unit 1)
 				)
@@
 		(dnp no)
 		(fields_autoplaced yes)
-		(property "Reference" "#PWR?"
+		(property "Reference" "#PWR0106"
 			(at 115.57 101.6 0)
 			(effects
@@
 			(project "multiplexI2C"
 				(path "/0c2d0c14-8850-4a30-bb78-b2f40cb442ba/872e59d9-aae9-4a0c-a438-0cad18134c8d"
-					(reference "#PWR?")
+					(reference "#PWR0106")
 					(unit 1)
 				)
@@
 		(on_board yes)
 		(dnp no)
-		(property "Reference" "C?"
+		(property "Reference" "C102"
 			(at 85.09 97.79 0)
 			(effects
@@
 			(project "multiplexI2C"
 				(path "/0c2d0c14-8850-4a30-bb78-b2f40cb442ba/872e59d9-aae9-4a0c-a438-0cad18134c8d"
-					(reference "C?")
+					(reference "C102")
 					(unit 1)
 				)
@@
 		(on_board yes)
 		(dnp no)
-		(property "Reference" "D?"
+		(property "Reference" "D101"
 			(at 144.78 124.46 0)
 			(effects
@@
 			(project "multiplexI2C"
 				(path "/0c2d0c14-8850-4a30-bb78-b2f40cb442ba/872e59d9-aae9-4a0c-a438-0cad18134c8d"
-					(reference "D?")
+					(reference "D101")
 					(unit 1)
 				)
@@
 		(on_board yes)
 		(dnp no)
-		(property "Reference" "C?"
+		(property "Reference" "C106"
 			(at 161.544 98.298 0)
 			(effects
@@
 			(project "multiplexI2C"
 				(path "/0c2d0c14-8850-4a30-bb78-b2f40cb442ba/872e59d9-aae9-4a0c-a438-0cad18134c8d"
-					(reference "C?")
+					(reference "C106")
 					(unit 1)
 				)
@@
 		(dnp no)
 		(fields_autoplaced yes)
-		(property "Reference" "C?"
+		(property "Reference" "C101"
 			(at 123.19 69.8499 0)
 			(effects
@@
 			(project "multiplexI2C"
 				(path "/0c2d0c14-8850-4a30-bb78-b2f40cb442ba/872e59d9-aae9-4a0c-a438-0cad18134c8d"
-					(reference "C?")
+					(reference "C101")
 					(unit 1)
 				)
@@
 		(dnp no)
 		(fields_autoplaced yes)
-		(property "Reference" "#PWR?"
+		(property "Reference" "#PWR0109"
 			(at 160.02 132.08 0)
 			(effects
@@
 			(project "multiplexI2C"
 				(path "/0c2d0c14-8850-4a30-bb78-b2f40cb442ba/872e59d9-aae9-4a0c-a438-0cad18134c8d"
-					(reference "#PWR?")
+					(reference "#PWR0109")
 					(unit 1)
 				)
@@
 		(dnp no)
 		(fields_autoplaced yes)
-		(property "Reference" "#PWR?"
+		(property "Reference" "#PWR0104"
 			(at 147.32 60.96 0)
 			(effects
@@
 			(project "multiplexI2C"
 				(path "/0c2d0c14-8850-4a30-bb78-b2f40cb442ba/872e59d9-aae9-4a0c-a438-0cad18134c8d"
-					(reference "#PWR?")
+					(reference "#PWR0104")
 					(unit 1)
 				)
@@
 		(on_board yes)
 		(dnp no)
-		(property "Reference" "C?"
+		(property "Reference" "C103"
 			(at 95.25 97.79 0)
 			(effects
@@
 			(project "multiplexI2C"
 				(path "/0c2d0c14-8850-4a30-bb78-b2f40cb442ba/872e59d9-aae9-4a0c-a438-0cad18134c8d"
-					(reference "C?")
+					(reference "C103")
 					(unit 1)
 				)

Commit message: th8-F411 2025-12 plus some cleanup post manufacturing.
Parts:
- added C107, C108: 10µF, ProjectLib:C_0402_1005Metric, symbol ProjectLib:C
Connections:
- net +3V3: now also C108.1
- net +5V: now also C107.1
- net GND: now also C107.2, C108.2
